Commit message: updated camera_link to oak_imu_frame in the robot description

File: ros2_ws/src/bringup/urdf/rover.urdf (robot description, URDF)
Before this commit: robot rover, 3 links, 2 joints
Links:
- removed link camera_link
- added link oak_imu_frame
Joints:
- joint base_to_camera: child camera_link -> oak_imu_frame

Commit message: pushing latest code for IMU fusion

File: ros2_ws/src/bringup/urdf/rover.urdf (robot description, URDF)
Before this commit: robot rover, 3 links, 2 joints
Links:
- removed link oak_imu_frame
- added link oak_parent_frame
Joints:
- joint base_to_camera: child oak_imu_frame -> oak_parent_frame; origin xyz=0 0.2159 0.1651 rpy=0 0 0 -> xyz=0 0.2159 0.1651 rpy=3.14159265359 0 0
