Commit message: added collision and inertial properties to urdf file

File: ros2_ws/src/rover_description/src/description/rover_description.urdf (robot description, URDF)
Before this commit: robot rover, 5 links, 4 joints
Links:
- link base_link: geometry collision box size=${base_length} ${base_width} ${base_height}; visual box size=${base_length} ${base_width} ${base_height}
- link front_caster: geometry collision sphere radius=${(wheel_radius+wheel_zoff-(base_height/2))}; visual sphere radius=${(wheel_radius+wheel_zoff-(base_height/2))}
- link laser: geometry collision cylinder length=${laser_length} radius=${laser_radius}; visual cylinder length=${laser_length} radius=${laser_radius}

Commit message: committing latest code for proper navigation

File: ros2_ws/src/rover_description/src/description/rover_description.urdf (robot description, URDF)
Before this commit: robot rover, 5 links, 4 joints
Joints:
- joint base_joint: child base_footprint -> base_link; origin xyz=0.0 0.0 ${-(wheel_radius+wheel_zoff)} rpy=0 0 0 -> xyz=0.0 0.0 ${wheel_radius + wheel_zoff} rpy=0 0 0; parent base_link -> base_footprint
